File: schematic/WirelessTeleInfo.sch (KiCad schematic (older format))
At the start: 8 parts, among them P2 TeleInfo, Q1 BS170, U1 LTV-814, U2 WeMos_mini

Commit message: Update Schematic for better stability
Parts:
- added R4: 100k, Resistors_SMD:R_0805_HandSoldering, symbol Device:R
Connections:
- net at Q1.1 (D), R1.2: now also U2.14 (D7); no longer U2.12 (D5)
- net at U2.15 (D8): now also R4.2
- net at U2.8 (Tx): now also R4.1
- no-connect marks 13 -> 11
Other:
- note added: "V2.2"
- note removed: "V2.1"
- moved on the sheet: C3, P2, Q1, R1, R2, R3, U1, U2

Commit message: Fix Schematic
Parts:
- R4: value 100k -> 10K
Changed lines of the file:
@@
 P 3950 900
 F 0 "R4" V 3850 900 50  0000 C CNN
-F 1 "100k" V 3950 900 50  0000 C CNN
+F 1 "10K" V 3950 900 50  0000 C CNN
 F 2 "Resistors_SMD:R_0805_HandSoldering" V 3880 900 50  0001 C CNN
 F 3 "~" H 3950 900 50  0001 C CNN
