File: schematic/WirelessTeleInfo.kicad_pcb (KiCad board)
At the start: 2 copper layers, 25.4 x 26 mm, 8 parts, among them P2 TeleInfo, Q1 BS170, U1 LTV-814, U2 WeMos_mini

Commit message: Update Schematic for better stability
Parts:
- added R4: 100k, Resistors_SMD:R_0805_HandSoldering, B.Cu at (43.8, 43.7)
- moved R1 3.94 mm to (40.0, 43.7)
- moved R3 3.70 mm to (36.2, 43.9)
Connections:
- U2 pad 12: Net-(Q1-Pad1) -> (no net)
- U2 pad 14: (no net) -> Net-(Q1-Pad1)
- U2 pad 15: (no net) -> Net-(R4-Pad2)
- U2 pad 8: (no net) -> Net-(R4-Pad1)
Routing:
- net Net-(R4-Pad1): track 0.00 -> 33.5 mm
- net Net-(Q1-Pad1): track 9.15 -> 18.9 mm
- net Net-(R4-Pad2): track 0.00 -> 4.60 mm
- net Net-(Q1-Pad2): track 16.9 -> 21.4 mm
- net GND: track 22.8 -> 24.8 mm
Other:
- board text added: "100K"
- board text added: "D7"
- board text added: "D8"
- board text added: "V2.2"
- board text removed: "D5"
- board text removed: "V2.1"

Commit message: Fix Schematic
Other:
- board text removed: "100K"
Changed lines of the file:
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@@
     (tags "resistor 0805")
     (attr smd)
-    (fp_text reference R3 (at 1.35 1.905 90) (layer B.SilkS)
+    (fp_text reference R3 (at 1.477 1.905 90) (layer B.SilkS)
       (effects (font (size 1 1) (thickness 0.15)) (justify mirror))
     )
@@
     (tags "resistor 0805")
     (attr smd)
-    (fp_text reference R4 (at -1.825 -1.905 270) (layer B.SilkS)
+    (fp_text reference R4 (at -1.444 -1.905 270) (layer B.SilkS)
       (effects (font (size 1 1) (thickness 0.15)) (justify mirror))
     )
@@
     (effects (font (size 1 1) (thickness 0.15)))
   )
-  (gr_text 100K (at 45.72 45.085 90) (layer B.SilkS)
+  (gr_text 10K (at 45.72 45.085 90) (layer B.SilkS)
     (effects (font (size 1 1) (thickness 0.15)) (justify mirror))
   )

Commit message: Cleanup and update schematic to KiCAD 8
Other:
- net class Default removed
